File: hw/board/UltrasonicMatrix.sch (EAGLE design)
At the start: 180 parts, among them IC1 7812L, U1 TC4427EOA, U10 TC4427EOA, U11 TC4427EOA, U12 TC4427EOA, U13 TC4427EOA, U14 TC4427EOA, U15 TC4427EOA, U16 TC4427EOA, U17 TC4427EOA, U18 TC4427EOA, U19 TC4427EOA, U2 TC4427EOA, U20 TC4427EOA, U21 TC4427EOA, U22 TC4427EOA, U23 TC4427EOA, U24 TC4427EOA, U25 TC4427EOA, U26 TC4427EOA, U27 TC4427EOA, U28 TC4427EOA, U29 TC4427EOA, U3 TC4427EOA, U30 TC4427EOA, U31 TC4427EOA, U32 TC4427EOA, U4 TC4427EOA, U5 TC4427EOA, U6 TC4427EOA, U7 TC4427EOA, U8 TC4427EOA, U9 TC4427EOA

Commit message: schematic done
Parts:
- removed SVI10: (no value), con-lstb:MA08-1
- added RESET: (no value), switch-omron:10-XX
- C65, C66: value (none) -> 100pF
- D1: value 1N4004 -> 1N4001
- SVI4: device con-lstb:MA18-2 -> con-lstb:MA08-1
- renumbered J1 to PWR_IN, SVI8 to SVI6, SVI9 to SVI5, SVJ8 to VIN_ENABLE
Connections:
- removed net 3V3: SVI10.5, SVO4.5
- removed net 5V: SVI10.4, SVI4.1, SVI7.1, SVI7.2, SVO4.4
- removed net V20: C1.1, C10.1, C12.1, C13.1, C14.1, C16.1, C17.1, C18.1, C2.1, C20.1, C21.1, C22.1, C24.1, C25.1, C26.1, C28.1, C29.1, C30.1, C32.1, C4.1, C5.1, C6.1, C65.1, C8.1, C9.1, D1.C, IC1.VI, U1.VDD, U10.VDD, U12.VDD, U13.VDD, U14.VDD, U16.VDD, U17.VDD, U18.VDD, U2.VDD, U20.VDD, U21.VDD, U22.VDD, U24.VDD, U25.VDD, U26.VDD, U28.VDD, U29.VDD, U30.VDD, U32.VDD, U4.VDD, U5.VDD, U6.VDD, U8.VDD, U9.VDD
- removed net V3: C11.1, C15.1, C19.1, C23.1, C27.1, C3.1, C31.1, C7.1, U11.VDD, U15.VDD, U19.VDD, U23.VDD, U27.VDD, U3.VDD, U31.VDD, U7.VDD
- removed net VCC: C33.1, C34.1, C35.1, C36.1, C37.1, C38.1, C39.1, C40.1, C41.1, C42.1, C43.1, C44.1, C45.1, C46.1, C47.1, C48.1, C49.1, C50.1, C51.1, C52.1, C53.1, C54.1, C55.1, C56.1, C57.1, C58.1, C59.1, C60.1, C61.1, C62.1, C63.1, C64.1
- new net +18V: C1.1, C10.1, C11.1, C12.1, C13.1, C14.1, C15.1, C16.1, C17.1, C18.1, C19.1, C2.1, C20.1, C21.1, C22.1, C23.1, C24.1, C25.1, C26.1, C27.1, C28.1, C29.1, C3.1, C30.1, C31.1, C32.1, C33.1, C34.1, C35.1, C36.1, C37.1, C38.1, C39.1, C4.1, C40.1, C41.1, C42.1, C43.1, C44.1, C45.1, C46.1, C47.1, C48.1, C49.1, C5.1, C50.1, C51.1, C52.1, C53.1, C54.1, C55.1, C56.1, C57.1, C58.1, C59.1, C6.1, C60.1, C61.1, C62.1, C63.1, C64.1, C65.1, C7.1, C8.1, C9.1, D1.C, IC1.VI, U1.VDD, U10.VDD, U11.VDD, U12.VDD, U13.VDD, U14.VDD, U15.VDD, U16.VDD, U17.VDD, U18.VDD, U19.VDD, U2.VDD, U20.VDD, U21.VDD, U22.VDD, U23.VDD, U24.VDD, U25.VDD, U26.VDD, U27.VDD, U28.VDD, U29.VDD, U3.VDD, U30.VDD, U31.VDD, U32.VDD, U4.VDD, U5.VDD, U6.VDD, U7.VDD, U8.VDD, U9.VDD
- new net +3V3: SVI4.5, SVO4.5
- new net +5V: SVI4.4, SVI7.1, SVI7.2, SVO4.4
- new net PD22: U$18.P0, U9.!OUT_A
- new net PD23: U$20.P0, U10.!OUT_A
- net GND: now also RESET.S, RESET.S1, SVI4.2, SVI4.3; no longer SVI10.2, SVI10.3, SVI4.35
- net IOREF: now also SVI4.7; no longer SVI10.7
- net PA23: now also U10.IN_A; no longer SVI4.3, U9.IN_B
- net PA24: now also U9.IN_B; no longer U10.IN_A
- net PA25: no longer SVI4.5
- net PA27: now also U12.IN_A; no longer SVI4.7, U11.IN_B
- net PA28: now also U11.IN_B; no longer U12.IN_A
- net PA29: no longer SVI4.9
- net PA31: now also U14.IN_A; no longer SVI4.11, U13.IN_B
- net PA32: now also U13.IN_B; no longer U14.IN_A
- net PA33: no longer SVI4.13
- net PA35: now also U16.IN_A; no longer SVI4.15, U15.IN_B
- net PA36: now also U15.IN_B; no longer U16.IN_A
- net PA37: no longer SVI4.17
- net PA39: now also U18.IN_A; no longer SVI4.19, U17.IN_B
- net PA40: now also U17.IN_B; no longer U18.IN_A
- net PA41: no longer SVI4.21
- net PA43: now also U20.IN_A; no longer SVI4.23, U19.IN_B
- net PA44: now also U19.IN_B; no longer U20.IN_A
- net PA45: no longer SVI4.25
- net PA47: now also U22.IN_A; no longer SVI4.27, U21.IN_B
- net PA48: now also U21.IN_B; no longer U22.IN_A
- net PA49: no longer SVI4.29
- net PA51: now also U24.IN_A; no longer SVI4.31, U23.IN_B
- net PA52: now also U23.IN_B; no longer U24.IN_A
- net PA53: no longer SVI4.33
- net PD24: now also U$17.P0, U9.!OUT_B; no longer U$20.P0, U10.!OUT_A
- net PD27: now also U$24.P0, U12.!OUT_A; no longer U$21.P0, U11.!OUT_B
- net PD28: now also U$21.P0, U11.!OUT_B; no longer U$24.P0, U12.!OUT_A
- net PD31: now also U$28.P0, U14.!OUT_A; no longer U$25.P0, U13.!OUT_B
- net PD32: now also U$25.P0, U13.!OUT_B; no longer U$28.P0, U14.!OUT_A
- net PD35: now also U$32.P0, U16.!OUT_A; no longer U$29.P0, U15.!OUT_B
- net PD36: now also U$29.P0, U15.!OUT_B; no longer U$32.P0, U16.!OUT_A
- net PD39: now also U$36.P0, U18.!OUT_A; no longer U$33.P0, U17.!OUT_B
- net PD40: now also U$33.P0, U17.!OUT_B; no longer U$36.P0, U18.!OUT_A
- net PD43: now also U$40.P0, U20.!OUT_A; no longer U$37.P0, U19.!OUT_B
- net PD44: now also U$37.P0, U19.!OUT_B; no longer U$40.P0, U20.!OUT_A
- net PD47: now also U$44.P0, U22.!OUT_A; no longer U$41.P0, U21.!OUT_B
- net PD48: now also U$41.P0, U21.!OUT_B; no longer U$44.P0, U22.!OUT_A
- net PD51: now also U$48.P0, U24.!OUT_A; no longer U$45.P0, U23.!OUT_B
- net PD52: now also U$45.P0, U23.!OUT_B; no longer U$48.P0, U24.!OUT_A
- net PD6: no longer U$18.P0, U9.!OUT_A
- net PD7: no longer U$17.P0, U9.!OUT_B
- net RESET: now also RESET.P, RESET.P1, SVI4.6; no longer SVI10.6
- net VIN: now also SVI4.1, VIN_ENABLE.3; no longer SVI10.1

Commit message: tracing
Parts:
- PWR_IN: value (none) -> DCJACK; device con-jack:JACK-PLUG0 -> DCJack:DCJACK
- U$1, U$10, U$11, U$12, U$13, U$14, U$15, U$16, U$17, U$18, U$19, U$2, U$20, U$21, U$22, U$23, U$24, U$25, U$26, U$27, U$28, U$29, U$3, U$30, U$31, U$32, U$33, U$34, U$35, U$36, U$37, U$38, U$39, U$4, U$40, U$41, U$42, U$43, U$44, U$45, U$46, U$47, U$48, U$49, U$5, U$50, U$51, U$52, U$53, U$54, U$55, U$56, U$57, U$58, U$59, U$6, U$60, U$61, U$62, U$63, U$64, U$7, U$9: device ultrasonic:TCT40-16 -> TCT40:TCT40-16
Connections:
- net GND: now also PWR_IN.GND; no longer PWR_IN.1, PWR_IN.2
- net N$1: now also PWR_IN.PWR; no longer PWR_IN.3

Commit message: more tracing
Connections:
- net PA22: now also U9.IN_B; no longer U9.IN_A
- net PA24: now also U9.IN_A; no longer U9.IN_B
- net PA26: now also U11.IN_B; no longer U11.IN_A
- net PA28: now also U11.IN_A; no longer U11.IN_B
- net PA30: now also U13.IN_B; no longer U13.IN_A
- net PA32: now also U13.IN_A; no longer U13.IN_B
- net PA34: now also U15.IN_B; no longer U15.IN_A
- net PA36: now also U15.IN_A; no longer U15.IN_B
- net PA38: now also U17.IN_B; no longer U17.IN_A
- net PA40: now also U17.IN_A; no longer U17.IN_B
- net PA42: now also U19.IN_B; no longer U19.IN_A
- net PA44: now also U19.IN_A; no longer U19.IN_B
- net PA46: now also U21.IN_B; no longer U21.IN_A
- net PA48: now also U21.IN_A; no longer U21.IN_B
- net PA50: now also U23.IN_B; no longer U23.IN_A
- net PA52: now also U23.IN_A; no longer U23.IN_B
- net PD22: now also U$17.P0, U9.!OUT_B; no longer U$18.P0, U9.!OUT_A
- net PD24: now also U$18.P0, U9.!OUT_A; no longer U$17.P0, U9.!OUT_B
- net PD26: now also U$21.P0, U11.!OUT_B; no longer U$22.P0, U11.!OUT_A
- net PD28: now also U$22.P0, U11.!OUT_A; no longer U$21.P0, U11.!OUT_B
- net PD30: now also U$25.P0, U13.!OUT_B; no longer U$26.P0, U13.!OUT_A
- net PD32: now also U$26.P0, U13.!OUT_A; no longer U$25.P0, U13.!OUT_B
- net PD34: now also U$29.P0, U15.!OUT_B; no longer U$30.P0, U15.!OUT_A
- net PD36: now also U$30.P0, U15.!OUT_A; no longer U$29.P0, U15.!OUT_B
- net PD38: now also U$33.P0, U17.!OUT_B; no longer U$34.P0, U17.!OUT_A
- net PD40: now also U$34.P0, U17.!OUT_A; no longer U$33.P0, U17.!OUT_B
- net PD42: now also U$37.P0, U19.!OUT_B; no longer U$38.P0, U19.!OUT_A
- net PD44: now also U$38.P0, U19.!OUT_A; no longer U$37.P0, U19.!OUT_B
- net PD46: now also U$41.P0, U21.!OUT_B; no longer U$42.P0, U21.!OUT_A
- net PD48: now also U$42.P0, U21.!OUT_A; no longer U$41.P0, U21.!OUT_B
- net PD50: now also U$45.P0, U23.!OUT_B; no longer U$46.P0, U23.!OUT_A
- net PD52: now also U$46.P0, U23.!OUT_A; no longer U$45.P0, U23.!OUT_B

Commit message: almost done
Connections:
- net PA6: now also U1.IN_B; no longer U1.IN_A
- net PA64: now also U30.IN_B; no longer U30.IN_A
- net PA65: now also U30.IN_A; no longer U30.IN_B
- net PA66: now also U31.IN_B; no longer U31.IN_A
- net PA67: now also U31.IN_A; no longer U31.IN_B
- net PA68: now also U32.IN_B; no longer U32.IN_A
- net PA69: now also U32.IN_A; no longer U32.IN_B
- net PA7: now also U1.IN_A; no longer U1.IN_B
- net PA8: now also U2.IN_B; no longer U2.IN_A
- net PA9: now also U2.IN_A; no longer U2.IN_B
- net PD6: now also U$3.P0, U1.!OUT_B; no longer U$4.P0, U1.!OUT_A
- net PD64: now also U$59.P0, U30.!OUT_B; no longer U$60.P0, U30.!OUT_A
- net PD65: now also U$60.P0, U30.!OUT_A; no longer U$59.P0, U30.!OUT_B
- net PD66: now also U$61.P0, U31.!OUT_B; no longer U$62.P0, U31.!OUT_A
- net PD67: now also U$62.P0, U31.!OUT_A; no longer U$61.P0, U31.!OUT_B
- net PD68: now also U$63.P0, U32.!OUT_B; no longer U$64.P0, U32.!OUT_A
- net PD69: now also U$64.P0, U32.!OUT_A; no longer U$63.P0, U32.!OUT_B
- net PD7: now also U$4.P0, U1.!OUT_A; no longer U$3.P0, U1.!OUT_B
- net PD8: now also U$5.P0, U2.!OUT_B; no longer U$6.P0, U2.!OUT_A
- net PD9: now also U$6.P0, U2.!OUT_A; no longer U$5.P0, U2.!OUT_B
Changed lines of the file:
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@@
 </segment>
 <segment>
-<pinref part="U1" gate="A" pin="IN_A"/>
-<wire x1="160.02" y1="134.62" x2="144.78" y2="134.62" width="0.1524" layer="91"/>
-<label x="147.32" y="134.62" size="1.778" layer="95"/>
+<pinref part="U1" gate="A" pin="IN_B"/>
+<wire x1="160.02" y1="132.08" x2="144.78" y2="132.08" width="0.1524" layer="91"/>
+<label x="147.32" y="132.08" size="1.778" layer="95"/>
 </segment>
 </net>
@@
 </segment>
 <segment>
-<pinref part="U1" gate="A" pin="IN_B"/>
-<wire x1="160.02" y1="132.08" x2="144.78" y2="132.08" width="0.1524" layer="91"/>
-<label x="147.32" y="132.08" size="1.778" layer="95"/>
+<pinref part="U1" gate="A" pin="IN_A"/>
+<wire x1="160.02" y1="134.62" x2="144.78" y2="134.62" width="0.1524" layer="91"/>
+<label x="147.32" y="134.62" size="1.778" layer="95"/>
 </segment>
 </net>
@@
 </segment>
 <segment>
-<pinref part="U2" gate="A" pin="IN_A"/>
-<wire x1="160.02" y1="88.9" x2="144.78" y2="88.9" width="0.1524" layer="91"/>
-<label x="147.32" y="88.9" size="1.778" layer="95"/>
+<pinref part="U2" gate="A" pin="IN_B"/>
+<wire x1="160.02" y1="86.36" x2="144.78" y2="86.36" width="0.1524" layer="91"/>
+<label x="147.32" y="86.36" size="1.778" layer="95"/>
 </segment>
 </net>
@@
 </segment>
 <segment>
-<pinref part="U2" gate="A" pin="IN_B"/>
-<wire x1="160.02" y1="86.36" x2="144.78" y2="86.36" width="0.1524" layer="91"/>
-<label x="147.32" y="86.36" size="1.778" layer="95"/>
+<pinref part="U2" gate="A" pin="IN_A"/>
+<wire x1="160.02" y1="88.9" x2="144.78" y2="88.9" width="0.1524" layer="91"/>
+<label x="147.32" y="88.9" size="1.778" layer="95"/>
 </segment>
 </net>
@@
 </segment>
 <segment>
-<pinref part="U32" gate="A" pin="IN_B"/>
-<wire x1="429.26" y1="-187.96" x2="414.02" y2="-187.96" width="0.1524" layer="91"/>
-<label x="416.56" y="-187.96" size="1.778" layer="95"/>
+<pinref part="U32" gate="A" pin="IN_A"/>
+<wire x1="429.26" y1="-185.42" x2="414.02" y2="-185.42" width="0.1524" layer="91"/>
+<label x="416.56" y="-185.42" size="1.778" layer="95"/>
 </segment>
 </net>
@@
 </segment>
 <segment>
-<pinref part="U30" gate="A" pin="IN_A"/>
-<wire x1="429.26" y1="-93.98" x2="414.02" y2="-93.98" width="0.1524" layer="91"/>
-<label x="416.56" y="-93.98" size="1.778" layer="95"/>
+<pinref part="U30" gate="A" pin="IN_B"/>
+<wire x1="429.26" y1="-96.52" x2="414.02" y2="-96.52" width="0.1524" layer="91"/>
+<label x="416.56" y="-96.52" size="1.778" layer="95"/>
 </segment>
 </net>
@@
 </segment>
 <segment>
-<pinref part="U30" gate="A" pin="IN_B"/>
-<wire x1="429.26" y1="-96.52" x2="414.02" y2="-96.52" width="0.1524" layer="91"/>
-<label x="416.56" y="-96.52" size="1.778" layer="95"/>
+<pinref part="U30" gate="A" pin="IN_A"/>
+<wire x1="429.26" y1="-93.98" x2="414.02" y2="-93.98" width="0.1524" layer="91"/>
+<label x="416.56" y="-93.98" size="1.778" layer="95"/>
 </segment>
 </net>
@@
 </segment>
 <segment>
-<pinref part="U31" gate="A" pin="IN_A"/>
-<wire x1="429.26" y1="-139.7" x2="414.02" y2="-139.7" width="0.1524" layer="91"/>
-<label x="416.56" y="-139.7" size="1.778" layer="95"/>
+<pinref part="U31" gate="A" pin="IN_B"/>
+<wire x1="429.26" y1="-142.24" x2="414.02" y2="-142.24" width="0.1524" layer="91"/>
+<label x="416.56" y="-142.24" size="1.778" layer="95"/>
 </segment>
 </net>
@@
 </segment>
 <segment>
-<pinref part="U31" gate="A" pin="IN_B"/>
-<wire x1="429.26" y1="-142.24" x2="414.02" y2="-142.24" width="0.1524" layer="91"/>
-<label x="416.56" y="-142.24" size="1.778" layer="95"/>
+<pinref part="U31" gate="A" pin="IN_A"/>
+<wire x1="429.26" y1="-139.7" x2="414.02" y2="-139.7" width="0.1524" layer="91"/>
+<label x="416.56" y="-139.7" size="1.778" layer="95"/>
 </segment>
 </net>
@@
 </segment>
 <segment>
-<pinref part="U32" gate="A" pin="IN_A"/>
-<wire x1="429.26" y1="-185.42" x2="414.02" y2="-185.42" width="0.1524" layer="91"/>
-<label x="416.56" y="-185.42" size="1.778" layer="95"/>
+<pinref part="U32" gate="A" pin="IN_B"/>
+<wire x1="429.26" y1="-187.96" x2="414.02" y2="-187.96" width="0.1524" layer="91"/>
+<label x="416.56" y="-187.96" size="1.778" layer="95"/>
 </segment>
 </net>
@@
 </segment>
 </net>
-<net name="PD6" class="4">
+<net name="PD7" class="4">
 <segment>
 <pinref part="U1" gate="A" pin="!OUT_A"/>
@@
 </segment>
 </net>
-<net name="PD7" class="4">
-<segment>
-<pinref part="U1" gate="A" pin="!OUT_B"/>
-<wire x1="195.58" y1="132.08" x2="210.82" y2="132.08" width="0.1524" layer="91"/>
-<wire x1="210.82" y1="132.08" x2="210.82" y2="124.46" width="0.1524" layer="91"/>
-<pinref part="U$3" gate="G$1" pin="P0"/>
-<wire x1="210.82" y1="124.46" x2="215.9" y2="124.46" width="0.1524" layer="91"/>
-<label x="200.66" y="132.08" size="1.778" layer="95"/>
-</segment>
-</net>
-<net name="PD8" class="4">
+<net name="PD9" class="4">
 <segment>
 <pinref part="U2" gate="A" pin="!OUT_A"/>
@@
 </segment>
 </net>
-<net name="PD9" class="4">
-<segment>
-<pinref part="U2" gate="A" pin="!OUT_B"/>
-<wire x1="195.58" y1="86.36" x2="210.82" y2="86.36" width="0.1524" layer="91"/>
-<wire x1="210.82" y1="86.36" x2="210.82" y2="78.74" width="0.1524" layer="91"/>
-<pinref part="U$5" gate="G$1" pin="P0"/>
-<wire x1="210.82" y1="78.74" x2="215.9" y2="78.74" width="0.1524" layer="91"/>
-<label x="200.66" y="86.36" size="1.778" layer="95"/>
-</segment>
-</net>
 <net name="PD10" class="4">
 <segment>
@@
 </segment>
 </net>
-<net name="PD64" class="4">
+<net name="PD65" class="4">
 <segment>
 <pinref part="U30" gate="A" pin="!OUT_A"/>
@@
 </segment>
 </net>
-<net name="PD65" class="4">
-<segment>
-<pinref part="U30" gate="A" pin="!OUT_B"/>
-<wire x1="464.82" y1="-96.52" x2="480.06" y2="-96.52" width="0.1524" layer="91"/>
-<wire x1="480.06" y1="-96.52" x2="480.06" y2="-104.14" width="0.1524" layer="91"/>
-<pinref part="U$59" gate="G$1" pin="P0"/>
-<wire x1="480.06" y1="-104.14" x2="485.14" y2="-104.14" width="0.1524" layer="91"/>
-<label x="469.9" y="-96.52" size="1.778" layer="95"/>
-</segment>
-</net>
-<net name="PD66" class="4">
+<net name="PD67" class="4">
 <segment>
 <pinref part="U31" gate="A" pin="!OUT_A"/>
@@
 </segment>
 </net>
-<net name="PD67" class="4">
-<segment>
-<pinref part="U31" gate="A" pin="!OUT_B"/>
-<wire x1="464.82" y1="-142.24" x2="480.06" y2="-142.24" width="0.1524" layer="91"/>
-<wire x1="480.06" y1="-142.24" x2="480.06" y2="-149.86" width="0.1524" layer="91"/>
-<pinref part="U$61" gate="G$1" pin="P0"/>
-<wire x1="480.06" y1="-149.86" x2="485.14" y2="-149.86" width="0.1524" layer="91"/>
-<label x="469.9" y="-142.24" size="1.778" layer="95"/>
-</segment>
-</net>
-<net name="PD68" class="4">
+<net name="PD69" class="4">
 <segment>
 <pinref part="U32" gate="A" pin="!OUT_A"/>
@@
 <wire x1="480.06" y1="-180.34" x2="485.14" y2="-180.34" width="0.1524" layer="91"/>
 <label x="469.9" y="-185.42" size="1.778" layer="95"/>
-</segment>
-</net>
-<net name="PD69" class="4">
-<segment>
-<pinref part="U32" gate="A" pin="!OUT_B"/>
-<wire x1="464.82" y1="-187.96" x2="480.06" y2="-187.96" width="0.1524" layer="91"/>
-<wire x1="480.06" y1="-187.96" x2="480.06" y2="-195.58" width="0.1524" layer="91"/>
-<pinref part="U$63" gate="G$1" pin="P0"/>
-<wire x1="480.06" y1="-195.58" x2="485.14" y2="-195.58" width="0.1524" layer="91"/>
-<label x="469.9" y="-187.96" size="1.778" layer="95"/>
 </segment>
 </net>
@@
 </segment>
 </net>
+<net name="PD6" class="4">
+<segment>
+<pinref part="U1" gate="A" pin="!OUT_B"/>
+<wire x1="195.58" y1="132.08" x2="210.82" y2="132.08" width="0.1524" layer="91"/>
+<wire x1="210.82" y1="132.08" x2="210.82" y2="124.46" width="0.1524" layer="91"/>
+<pinref part="U$3" gate="G$1" pin="P0"/>
+<wire x1="210.82" y1="124.46" x2="215.9" y2="124.46" width="0.1524" layer="91"/>
+<label x="200.66" y="132.08" size="1.778" layer="95"/>
+</segment>
+</net>
+<net name="PD8" class="4">
+<segment>
+<pinref part="U2" gate="A" pin="!OUT_B"/>
+<wire x1="195.58" y1="86.36" x2="210.82" y2="86.36" width="0.1524" layer="91"/>
+<wire x1="210.82" y1="86.36" x2="210.82" y2="78.74" width="0.1524" layer="91"/>
+<pinref part="U$5" gate="G$1" pin="P0"/>
+<wire x1="210.82" y1="78.74" x2="215.9" y2="78.74" width="0.1524" layer="91"/>
+<label x="200.66" y="86.36" size="1.778" layer="95"/>
+</segment>
+</net>
+<net name="PD64" class="4">
+<segment>
+<pinref part="U30" gate="A" pin="!OUT_B"/>
+<wire x1="464.82" y1="-96.52" x2="480.06" y2="-96.52" width="0.1524" layer="91"/>
+<wire x1="480.06" y1="-96.52" x2="480.06" y2="-104.14" width="0.1524" layer="91"/>
+<pinref part="U$59" gate="G$1" pin="P0"/>
+<wire x1="480.06" y1="-104.14" x2="485.14" y2="-104.14" width="0.1524" layer="91"/>
+<label x="469.9" y="-96.52" size="1.778" layer="95"/>
+</segment>
+</net>
+<net name="PD66" class="4">
+<segment>
+<pinref part="U31" gate="A" pin="!OUT_B"/>
+<wire x1="464.82" y1="-142.24" x2="480.06" y2="-142.24" width="0.1524" layer="91"/>
+<wire x1="480.06" y1="-142.24" x2="480.06" y2="-149.86" width="0.1524" layer="91"/>
+<pinref part="U$61" gate="G$1" pin="P0"/>
+<wire x1="480.06" y1="-149.86" x2="485.14" y2="-149.86" width="0.1524" layer="91"/>
+<label x="469.9" y="-142.24" size="1.778" layer="95"/>
+</segment>
+</net>
+<net name="PD68" class="4">
+<segment>
+<pinref part="U32" gate="A" pin="!OUT_B"/>
+<wire x1="464.82" y1="-187.96" x2="480.06" y2="-187.96" width="0.1524" layer="91"/>
+<wire x1="480.06" y1="-187.96" x2="480.06" y2="-195.58" width="0.1524" layer="91"/>
+<pinref part="U$63" gate="G$1" pin="P0"/>
+<wire x1="480.06" y1="-195.58" x2="485.14" y2="-195.58" width="0.1524" layer="91"/>
+<label x="469.9" y="-187.96" size="1.778" layer="95"/>
+</segment>
+</net>
