File: hw/board/UltrasonicMatrix.sch (EAGLE design)
At the start: 180 parts, among them IC1 7812L, U1 TC4427EOA, U10 TC4427EOA, U11 TC4427EOA, U12 TC4427EOA, U13 TC4427EOA, U14 TC4427EOA, U15 TC4427EOA, U16 TC4427EOA, U17 TC4427EOA, U18 TC4427EOA, U19 TC4427EOA, U2 TC4427EOA, U20 TC4427EOA, U21 TC4427EOA, U22 TC4427EOA, U23 TC4427EOA, U24 TC4427EOA, U25 TC4427EOA, U26 TC4427EOA, U27 TC4427EOA, U28 TC4427EOA, U29 TC4427EOA, U3 TC4427EOA, U30 TC4427EOA, U31 TC4427EOA, U32 TC4427EOA, U4 TC4427EOA, U5 TC4427EOA, U6 TC4427EOA, U7 TC4427EOA, U8 TC4427EOA, U9 TC4427EOA

Commit message: more on board layout
Connections:
- net PA56: now also U26.IN_B; no longer U26.IN_A
- net PA57: now also U26.IN_A; no longer U26.IN_B
- net PA58: now also U27.IN_B; no longer U27.IN_A
- net PA59: now also U27.IN_A; no longer U27.IN_B
- net PA60: now also U28.IN_B; no longer U28.IN_A
- net PA61: now also U28.IN_A; no longer U28.IN_B
- net PA62: now also U29.IN_B; no longer U29.IN_A
- net PA63: now also U29.IN_A; no longer U29.IN_B
- net PD56: now also U$51.P0, U26.!OUT_B; no longer U$52.P0, U26.!OUT_A
- net PD57: now also U$52.P0, U26.!OUT_A; no longer U$51.P0, U26.!OUT_B
- net PD58: now also U$53.P0, U27.!OUT_B; no longer U$54.P0, U27.!OUT_A
- net PD59: now also U$54.P0, U27.!OUT_A; no longer U$53.P0, U27.!OUT_B
- net PD60: now also U$55.P0, U28.!OUT_B; no longer U$56.P0, U28.!OUT_A
- net PD61: now also U$56.P0, U28.!OUT_A; no longer U$55.P0, U28.!OUT_B
- net PD62: now also U$57.P0, U29.!OUT_B; no longer U$58.P0, U29.!OUT_A
- net PD63: now also U$58.P0, U29.!OUT_A; no longer U$57.P0, U29.!OUT_B
Changed lines of the file:
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@@
 </variantdefs>
 <classes>
-<class number="0" name="default" width="0.4572" drill="0.254">
+<class number="0" name="default" width="0.508" drill="0.254">
 <clearance class="0" value="0.205"/>
 </class>
@@
 <class number="5" name="GND" width="0.762" drill="0">
 </class>
-<class number="6" name="+12V" width="1.27" drill="0">
+<class number="6" name="+12V" width="1.016" drill="0">
 </class>
 </classes>
@@
 </segment>
 <segment>
-<pinref part="U26" gate="A" pin="IN_A"/>
-<wire x1="429.26" y1="88.9" x2="414.02" y2="88.9" width="0.1524" layer="91"/>
-<label x="416.56" y="88.9" size="1.778" layer="95"/>
+<pinref part="U26" gate="A" pin="IN_B"/>
+<wire x1="429.26" y1="86.36" x2="414.02" y2="86.36" width="0.1524" layer="91"/>
+<label x="416.56" y="86.36" size="1.778" layer="95"/>
 </segment>
 </net>
@@
 </segment>
 <segment>
-<pinref part="U26" gate="A" pin="IN_B"/>
-<wire x1="429.26" y1="86.36" x2="414.02" y2="86.36" width="0.1524" layer="91"/>
-<label x="416.56" y="86.36" size="1.778" layer="95"/>
+<pinref part="U26" gate="A" pin="IN_A"/>
+<wire x1="429.26" y1="88.9" x2="414.02" y2="88.9" width="0.1524" layer="91"/>
+<label x="416.56" y="88.9" size="1.778" layer="95"/>
 </segment>
 </net>
@@
 </segment>
 <segment>
-<pinref part="U27" gate="A" pin="IN_A"/>
-<wire x1="429.26" y1="43.18" x2="414.02" y2="43.18" width="0.1524" layer="91"/>
-<label x="416.56" y="43.18" size="1.778" layer="95"/>
+<pinref part="U27" gate="A" pin="IN_B"/>
+<wire x1="429.26" y1="40.64" x2="414.02" y2="40.64" width="0.1524" layer="91"/>
+<label x="416.56" y="40.64" size="1.778" layer="95"/>
 </segment>
 </net>
@@
 </segment>
 <segment>
-<pinref part="U27" gate="A" pin="IN_B"/>
-<wire x1="429.26" y1="40.64" x2="414.02" y2="40.64" width="0.1524" layer="91"/>
-<label x="416.56" y="40.64" size="1.778" layer="95"/>
+<pinref part="U27" gate="A" pin="IN_A"/>
+<wire x1="429.26" y1="43.18" x2="414.02" y2="43.18" width="0.1524" layer="91"/>
+<label x="416.56" y="43.18" size="1.778" layer="95"/>
 </segment>
 </net>
@@
 </segment>
 <segment>
-<pinref part="U28" gate="A" pin="IN_A"/>
-<wire x1="429.26" y1="-2.54" x2="414.02" y2="-2.54" width="0.1524" layer="91"/>
-<label x="416.56" y="-2.54" size="1.778" layer="95"/>
+<pinref part="U28" gate="A" pin="IN_B"/>
+<wire x1="429.26" y1="-5.08" x2="414.02" y2="-5.08" width="0.1524" layer="91"/>
+<label x="416.56" y="-5.08" size="1.778" layer="95"/>
 </segment>
 </net>
@@
 </segment>
 <segment>
-<pinref part="U28" gate="A" pin="IN_B"/>
-<wire x1="429.26" y1="-5.08" x2="414.02" y2="-5.08" width="0.1524" layer="91"/>
-<label x="416.56" y="-5.08" size="1.778" layer="95"/>
+<pinref part="U28" gate="A" pin="IN_A"/>
+<wire x1="429.26" y1="-2.54" x2="414.02" y2="-2.54" width="0.1524" layer="91"/>
+<label x="416.56" y="-2.54" size="1.778" layer="95"/>
 </segment>
 </net>
@@
 </segment>
 <segment>
-<pinref part="U29" gate="A" pin="IN_A"/>
-<wire x1="429.26" y1="-48.26" x2="414.02" y2="-48.26" width="0.1524" layer="91"/>
-<label x="416.56" y="-48.26" size="1.778" layer="95"/>
+<pinref part="U29" gate="A" pin="IN_B"/>
+<wire x1="429.26" y1="-50.8" x2="414.02" y2="-50.8" width="0.1524" layer="91"/>
+<label x="416.56" y="-50.8" size="1.778" layer="95"/>
 </segment>
 </net>
@@
 </segment>
 <segment>
-<pinref part="U29" gate="A" pin="IN_B"/>
-<wire x1="429.26" y1="-50.8" x2="414.02" y2="-50.8" width="0.1524" layer="91"/>
-<label x="416.56" y="-50.8" size="1.778" layer="95"/>
+<pinref part="U29" gate="A" pin="IN_A"/>
+<wire x1="429.26" y1="-48.26" x2="414.02" y2="-48.26" width="0.1524" layer="91"/>
+<label x="416.56" y="-48.26" size="1.778" layer="95"/>
 </segment>
 </net>
@@
 </segment>
 </net>
-<net name="PD54" class="4">
-<segment>
-<pinref part="U25" gate="A" pin="!OUT_A"/>
-<wire x1="464.82" y1="134.62" x2="480.06" y2="134.62" width="0.1524" layer="91"/>
-<wire x1="480.06" y1="134.62" x2="480.06" y2="139.7" width="0.1524" layer="91"/>
-<pinref part="U$50" gate="G$1" pin="P0"/>
-<wire x1="480.06" y1="139.7" x2="485.14" y2="139.7" width="0.1524" layer="91"/>
-<label x="469.9" y="134.62" size="1.778" layer="95"/>
-</segment>
-</net>
-<net name="PD55" class="4">
-<segment>
-<pinref part="U25" gate="A" pin="!OUT_B"/>
-<wire x1="464.82" y1="132.08" x2="480.06" y2="132.08" width="0.1524" layer="91"/>
-<wire x1="480.06" y1="132.08" x2="480.06" y2="124.46" width="0.1524" layer="91"/>
-<pinref part="U$49" gate="G$1" pin="P0"/>
-<wire x1="480.06" y1="124.46" x2="485.14" y2="124.46" width="0.1524" layer="91"/>
-<label x="469.9" y="132.08" size="1.778" layer="95"/>
-</segment>
-</net>
-<net name="PD56" class="4">
+<net name="PD57" class="4">
 <segment>
 <pinref part="U26" gate="A" pin="!OUT_A"/>
@@
 </segment>
 </net>
-<net name="PD57" class="4">
-<segment>
-<pinref part="U26" gate="A" pin="!OUT_B"/>
-<wire x1="464.82" y1="86.36" x2="480.06" y2="86.36" width="0.1524" layer="91"/>
-<wire x1="480.06" y1="86.36" x2="480.06" y2="78.74" width="0.1524" layer="91"/>
-<pinref part="U$51" gate="G$1" pin="P0"/>
-<wire x1="480.06" y1="78.74" x2="485.14" y2="78.74" width="0.1524" layer="91"/>
-<label x="469.9" y="86.36" size="1.778" layer="95"/>
-</segment>
-</net>
-<net name="PD58" class="4">
+<net name="PD59" class="4">
 <segment>
 <pinref part="U27" gate="A" pin="!OUT_A"/>
@@
 </segment>
 </net>
-<net name="PD59" class="4">
-<segment>
-<pinref part="U27" gate="A" pin="!OUT_B"/>
-<wire x1="464.82" y1="40.64" x2="480.06" y2="40.64" width="0.1524" layer="91"/>
-<wire x1="480.06" y1="40.64" x2="480.06" y2="33.02" width="0.1524" layer="91"/>
-<pinref part="U$53" gate="G$1" pin="P0"/>
-<wire x1="480.06" y1="33.02" x2="485.14" y2="33.02" width="0.1524" layer="91"/>
-<label x="469.9" y="40.64" size="1.778" layer="95"/>
-</segment>
-</net>
-<net name="PD60" class="4">
+<net name="PD61" class="4">
 <segment>
 <pinref part="U28" gate="A" pin="!OUT_A"/>
@@
 </segment>
 </net>
-<net name="PD61" class="4">
-<segment>
-<pinref part="U28" gate="A" pin="!OUT_B"/>
-<wire x1="464.82" y1="-5.08" x2="480.06" y2="-5.08" width="0.1524" layer="91"/>
-<wire x1="480.06" y1="-5.08" x2="480.06" y2="-12.7" width="0.1524" layer="91"/>
-<pinref part="U$55" gate="G$1" pin="P0"/>
-<wire x1="480.06" y1="-12.7" x2="485.14" y2="-12.7" width="0.1524" layer="91"/>
-<label x="469.9" y="-5.08" size="1.778" layer="95"/>
-</segment>
-</net>
-<net name="PD62" class="4">
+<net name="PD63" class="4">
 <segment>
 <pinref part="U29" gate="A" pin="!OUT_A"/>
@@
 </segment>
 </net>
-<net name="PD63" class="4">
-<segment>
-<pinref part="U29" gate="A" pin="!OUT_B"/>
-<wire x1="464.82" y1="-50.8" x2="480.06" y2="-50.8" width="0.1524" layer="91"/>
-<wire x1="480.06" y1="-50.8" x2="480.06" y2="-58.42" width="0.1524" layer="91"/>
-<pinref part="U$57" gate="G$1" pin="P0"/>
-<wire x1="480.06" y1="-58.42" x2="485.14" y2="-58.42" width="0.1524" layer="91"/>
-<label x="469.9" y="-50.8" size="1.778" layer="95"/>
-</segment>
-</net>
 <net name="PD65" class="4">
 <segment>
@@
 </segment>
 </net>
+<net name="PD58" class="4">
+<segment>
+<pinref part="U27" gate="A" pin="!OUT_B"/>
+<wire x1="464.82" y1="40.64" x2="480.06" y2="40.64" width="0.1524" layer="91"/>
+<wire x1="480.06" y1="40.64" x2="480.06" y2="33.02" width="0.1524" layer="91"/>
+<pinref part="U$53" gate="G$1" pin="P0"/>
+<wire x1="480.06" y1="33.02" x2="485.14" y2="33.02" width="0.1524" layer="91"/>
+<label x="469.9" y="40.64" size="1.778" layer="95"/>
+</segment>
+</net>
+<net name="PD60" class="4">
+<segment>
+<pinref part="U28" gate="A" pin="!OUT_B"/>
+<wire x1="464.82" y1="-5.08" x2="480.06" y2="-5.08" width="0.1524" layer="91"/>
+<wire x1="480.06" y1="-5.08" x2="480.06" y2="-12.7" width="0.1524" layer="91"/>
+<pinref part="U$55" gate="G$1" pin="P0"/>
+<wire x1="480.06" y1="-12.7" x2="485.14" y2="-12.7" width="0.1524" layer="91"/>
+<label x="469.9" y="-5.08" size="1.778" layer="95"/>
+</segment>
+</net>
+<net name="PD62" class="4">
+<segment>
+<pinref part="U29" gate="A" pin="!OUT_B"/>
+<wire x1="464.82" y1="-50.8" x2="480.06" y2="-50.8" width="0.1524" layer="91"/>
+<wire x1="480.06" y1="-50.8" x2="480.06" y2="-58.42" width="0.1524" layer="91"/>
+<pinref part="U$57" gate="G$1" pin="P0"/>
+<wire x1="480.06" y1="-58.42" x2="485.14" y2="-58.42" width="0.1524" layer="91"/>
+<label x="469.9" y="-50.8" size="1.778" layer="95"/>
+</segment>
+</net>
+<net name="PD54" class="4">
+<segment>
+<pinref part="U25" gate="A" pin="!OUT_A"/>
+<wire x1="464.82" y1="134.62" x2="480.06" y2="134.62" width="0.1524" layer="91"/>
+<wire x1="480.06" y1="134.62" x2="480.06" y2="139.7" width="0.1524" layer="91"/>
+<pinref part="U$50" gate="G$1" pin="P0"/>
+<wire x1="480.06" y1="139.7" x2="485.14" y2="139.7" width="0.1524" layer="91"/>
+<label x="469.9" y="134.62" size="1.778" layer="95"/>
+</segment>
+</net>
+<net name="PD56" class="4">
+<segment>
+<pinref part="U26" gate="A" pin="!OUT_B"/>
+<wire x1="464.82" y1="86.36" x2="480.06" y2="86.36" width="0.1524" layer="91"/>
+<wire x1="480.06" y1="86.36" x2="480.06" y2="78.74" width="0.1524" layer="91"/>
+<pinref part="U$51" gate="G$1" pin="P0"/>
+<wire x1="480.06" y1="78.74" x2="485.14" y2="78.74" width="0.1524" layer="91"/>
+<label x="469.9" y="86.36" size="1.778" layer="95"/>
+</segment>
+</net>
+<net name="PD55" class="4">
+<segment>
+<pinref part="U25" gate="A" pin="!OUT_B"/>
+<wire x1="464.82" y1="132.08" x2="480.06" y2="132.08" width="0.1524" layer="91"/>
+<wire x1="480.06" y1="132.08" x2="480.06" y2="124.46" width="0.1524" layer="91"/>
+<pinref part="U$49" gate="G$1" pin="P0"/>
+<wire x1="480.06" y1="124.46" x2="485.14" y2="124.46" width="0.1524" layer="91"/>
+<label x="469.9" y="132.08" size="1.778" layer="95"/>
+</segment>
+</net>

Commit message: Board completed
Parts:
- U$8: device ultrasonic:TCT40-16 -> TCT40:TCT40-16
Changed lines of the file:
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@@
 <part name="GND11" library="supply1" library_urn="urn:adsk.eagle:library:371" deviceset="GND" device=""/>
 <part name="U$7" library="TCT40" deviceset="TCT40-16" device=""/>
-<part name="U$8" library="ultrasonic" deviceset="TCT40-16" device=""/>
+<part name="U$8" library="TCT40" deviceset="TCT40-16" device=""/>
 <part name="U4" library="TC4427EOA" deviceset="TC4427EOA" device=""/>
 <part name="V8" library="supply1" library_urn="urn:adsk.eagle:library:371" deviceset="+18V" device="" value="V20"/>
@@
 </sheet>
 </sheets>
+<errors>
+</errors>
 </schematic>
 </drawing>
