File: hw/board/UltrasonicMatrix.brd (EAGLE design)
At the start: 142 x 142 mm, 180 parts, among them IC1 7812L, U1 TC4427EOA, U10 TC4427EOA, U11 TC4427EOA, U12 TC4427EOA, U13 TC4427EOA, U14 TC4427EOA, U15 TC4427EOA, U16 TC4427EOA, U17 TC4427EOA, U18 TC4427EOA, U19 TC4427EOA, U2 TC4427EOA, U20 TC4427EOA, U21 TC4427EOA, U22 TC4427EOA, U23 TC4427EOA, U24 TC4427EOA, U25 TC4427EOA, U26 TC4427EOA, U27 TC4427EOA, U28 TC4427EOA, U29 TC4427EOA, U3 TC4427EOA, U30 TC4427EOA, U31 TC4427EOA, U32 TC4427EOA, U4 TC4427EOA, U5 TC4427EOA, U6 TC4427EOA, U7 TC4427EOA, U8 TC4427EOA, U9 TC4427EOA

Commit message: schematic done
Parts:
- removed J1: (no value), con-jack:SPC4077
- removed SVI10, SVI8, SVI9: (no value), con-lstb:MA08-1
- removed SVJ8: (no value), con-lstb:MA03-1
- added PWR_IN: (no value), con-jack:SPC4077
- added RESET: (no value), switch-omron:B3F-10XX
- added SVI5, SVI6: (no value), con-lstb:MA08-1
- added VIN_ENABLE: (no value), con-lstb:MA03-1
- C65, C66: value (none) -> 100pF
- D1: value 1N4004 -> 1N4001
- SVI4: device con-lstb:MA18-2 -> con-lstb:MA08-1
- moved U5 327.5 mm to (197.9, 39.4)
- moved U6 327.5 mm to (185.2, 39.4)
- moved U7 327.5 mm to (172.5, 39.4)
- moved U8 327.5 mm to (159.8, 39.4)
- moved U$19 288.3 mm to (134.5, 32.5)
- moved SVO1 288.1 mm to (113.2, 56.2), turned to 90 degrees
- moved U$20 287.8 mm to (117.5, 32.5), turned to 180 degrees
- moved U1 266.2 mm to (194.3, 78.7)
- moved U2 266.2 mm to (181.6, 78.7)
- moved U3 266.2 mm to (168.9, 78.7)
- moved U4 266.2 mm to (156.2, 78.7)
- moved SVI3 262.7 mm to (107.6, 103.4), turned to 90 degrees
- moved U9 260.3 mm to (89.9, 131.1)
- moved U$28 239.1 mm to (100.5, 15.5), turned to 90 degrees
- moved U21 233.8 mm to (71.6, 100.6)
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Connections:
- removed net 3V3: SVI10.5, SVO4.5
- removed net 5V: SVI10.4, SVI4.1, SVI7.1, SVI7.2, SVO4.4
- removed net V20: C1.1, C10.1, C12.1, C13.1, C14.1, C16.1, C17.1, C18.1, C2.1, C20.1, C21.1, C22.1, C24.1, C25.1, C26.1, C28.1, C29.1, C30.1, C32.1, C4.1, C5.1, C6.1, C65.1, C8.1, C9.1, D1.C, IC1.3, U1.6, U10.6, U12.6, U13.6, U14.6, U16.6, U17.6, U18.6, U2.6, U20.6, U21.6, U22.6, U24.6, U25.6, U26.6, U28.6, U29.6, U30.6, U32.6, U4.6, U5.6, U6.6, U8.6, U9.6
- removed net V3: C11.1, C15.1, C19.1, C23.1, C27.1, C3.1, C31.1, C7.1, U11.6, U15.6, U19.6, U23.6, U27.6, U3.6, U31.6, U7.6
- removed net VCC: C33.1, C34.1, C35.1, C36.1, C37.1, C38.1, C39.1, C40.1, C41.1, C42.1, C43.1, C44.1, C45.1, C46.1, C47.1, C48.1, C49.1, C50.1, C51.1, C52.1, C53.1, C54.1, C55.1, C56.1, C57.1, C58.1, C59.1, C60.1, C61.1, C62.1, C63.1, C64.1
- new net +18V: C1.1, C10.1, C11.1, C12.1, C13.1, C14.1, C15.1, C16.1, C17.1, C18.1, C19.1, C2.1, C20.1, C21.1, C22.1, C23.1, C24.1, C25.1, C26.1, C27.1, C28.1, C29.1, C3.1, C30.1, C31.1, C32.1, C33.1, C34.1, C35.1, C36.1, C37.1, C38.1, C39.1, C4.1, C40.1, C41.1, C42.1, C43.1, C44.1, C45.1, C46.1, C47.1, C48.1, C49.1, C5.1, C50.1, C51.1, C52.1, C53.1, C54.1, C55.1, C56.1, C57.1, C58.1, C59.1, C6.1, C60.1, C61.1, C62.1, C63.1, C64.1, C65.1, C7.1, C8.1, C9.1, D1.C, IC1.3, U1.6, U10.6, U11.6, U12.6, U13.6, U14.6, U15.6, U16.6, U17.6, U18.6, U19.6, U2.6, U20.6, U21.6, U22.6, U23.6, U24.6, U25.6, U26.6, U27.6, U28.6, U29.6, U3.6, U30.6, U31.6, U32.6, U4.6, U5.6, U6.6, U7.6, U8.6, U9.6
- new net +3V3: SVI4.5, SVO4.5
- new net +5V: SVI4.4, SVI7.1, SVI7.2, SVO4.4
- new net PD22: U$18.P0, U9.7
- new net PD23: U$20.P0, U10.7
- net GND: now also PWR_IN.1, PWR_IN.2, RESET.1, RESET.2, SVI4.2, SVI4.3; no longer J1.1, J1.2, SVI10.2, SVI10.3, SVI4.35
- net IOREF: now also SVI4.7; no longer SVI10.7
- net N$1: now also PWR_IN.3; no longer J1.3
- net N$4: now also VIN_ENABLE.1; no longer SVJ8.1
- net PA23: now also U10.2; no longer SVI4.3, U9.4
- net PA24: now also U9.4; no longer U10.2
- net PA25: no longer SVI4.5
- net PA27: now also U12.2; no longer SVI4.7, U11.4
- net PA28: now also U11.4; no longer U12.2
- net PA29: no longer SVI4.9
- net PA31: now also U14.2; no longer SVI4.11, U13.4
- net PA32: now also U13.4; no longer U14.2
- net PA33: no longer SVI4.13
- net PA35: now also U16.2; no longer SVI4.15, U15.4
- net PA36: now also U15.4; no longer U16.2
- net PA37: no longer SVI4.17
- net PA39: now also U18.2; no longer SVI4.19, U17.4
- net PA40: now also U17.4; no longer U18.2
- net PA41: no longer SVI4.21
- net PA43: now also U20.2; no longer SVI4.23, U19.4
- net PA44: now also U19.4; no longer U20.2
- net PA45: no longer SVI4.25
- net PA47: now also U22.2; no longer SVI4.27, U21.4
- net PA48: now also U21.4; no longer U22.2
- net PA49: no longer SVI4.29
- net PA51: now also U24.2; no longer SVI4.31, U23.4
- net PA52: now also U23.4; no longer U24.2
- net PA53: no longer SVI4.33
- net PA54: now also SVI5.8; no longer SVI9.8
- net PA55: now also SVI5.7; no longer SVI9.7
- net PA56: now also SVI5.6; no longer SVI9.6
- net PA57: now also SVI5.5; no longer SVI9.5
- net PA58: now also SVI5.4; no longer SVI9.4
- net PA59: now also SVI5.3; no longer SVI9.3
- net PA60: now also SVI5.2; no longer SVI9.2
- net PA61: now also SVI5.1; no longer SVI9.1
- net PA62: now also SVI6.8; no longer SVI8.8
- net PA63: now also SVI6.7; no longer SVI8.7
- net PA64: now also SVI6.6; no longer SVI8.6
- net PA65: now also SVI6.5; no longer SVI8.5
- net PA66: now also SVI6.4; no longer SVI8.4
- net PA67: now also SVI6.3; no longer SVI8.3
- net PA68: now also SVI6.2; no longer SVI8.2
- net PA69: now also SVI6.1; no longer SVI8.1
- net PD24: now also U$17.P0, U9.5; no longer U$20.P0, U10.7
- net PD27: now also U$24.P0, U12.7; no longer U$21.P0, U11.5
- net PD28: now also U$21.P0, U11.5; no longer U$24.P0, U12.7
- net PD31: now also U$28.P0, U14.7; no longer U$25.P0, U13.5
- net PD32: now also U$25.P0, U13.5; no longer U$28.P0, U14.7
- net PD35: now also U$32.P0, U16.7; no longer U$29.P0, U15.5
- net PD36: now also U$29.P0, U15.5; no longer U$32.P0, U16.7
- net PD39: now also U$36.P0, U18.7; no longer U$33.P0, U17.5
- net PD40: now also U$33.P0, U17.5; no longer U$36.P0, U18.7
- net PD43: now also U$40.P0, U20.7; no longer U$37.P0, U19.5
- net PD44: now also U$37.P0, U19.5; no longer U$40.P0, U20.7
- net PD47: now also U$44.P0, U22.7; no longer U$41.P0, U21.5
- net PD48: now also U$41.P0, U21.5; no longer U$44.P0, U22.7
- net PD51: now also U$48.P0, U24.7; no longer U$45.P0, U23.5
- net PD52: now also U$45.P0, U23.5; no longer U$48.P0, U24.7
- net PD6: no longer U$18.P0, U9.7
- net PD7: no longer U$17.P0, U9.5
- net RESET: now also RESET.3, RESET.4, SVI4.6; no longer SVI10.6
- net VIN: now also SVI4.1, VIN_ENABLE.2, VIN_ENABLE.3; no longer SVI10.1, SVJ8.2
Other:
- board size 142 x 142 mm -> 150 x 150 mm
- board text added: "18VDC"
- board text added: "OFF"
- board text added: "ON"

Commit message: tracing
Parts:
- PWR_IN: value (none) -> DCJACK; device con-jack:SPC4077 -> DCJack:DCJACK
- U$1, U$10, U$11, U$12, U$13, U$14, U$15, U$16, U$17, U$18, U$19, U$2, U$20, U$21, U$22, U$23, U$24, U$25, U$26, U$27, U$28, U$29, U$3, U$30, U$31, U$32, U$33, U$34, U$35, U$36, U$37, U$38, U$39, U$4, U$40, U$41, U$42, U$43, U$44, U$45, U$46, U$47, U$48, U$49, U$5, U$50, U$51, U$52, U$53, U$54, U$55, U$56, U$57, U$58, U$59, U$6, U$60, U$61, U$62, U$63, U$64, U$7, U$9: device ultrasonic:TCT40-16 -> TCT40:TCT40-16
- moved U$39 53.8 mm to (15.5, 15.5), turned to 90 degrees
- moved U$43 38.0 mm to (66.5, 32.5), turned to 0 degrees
- moved U$44 38.0 mm to (49.5, 32.5), turned to 180 degrees
- moved U22 37.3 mm to (58.1, 25.9), turned to 90 degrees
- moved U20 37.1 mm to (23.4, 11.5), turned to 270 degrees
- moved U$40 24.0 mm to (32.5, 15.5), turned to 90 degrees
- moved U$32 18.0 mm to (82.5, 32.5), turned to 180 degrees
- moved U$31 17.0 mm to (100.5, 32.5), turned to 0 degrees
- moved U16 3.06 mm to (91.6, 26.9), turned to 90 degrees
- moved PWR_IN 1.71 mm to (12.2, 138.7), turned to 0 degrees
- moved SVI1 0.76 mm to (107.6, 57.0)
- moved SVI2 0.76 mm to (107.6, 79.8)
- moved SVI3 0.76 mm to (107.6, 104.2)
- moved SVI4 0.76 mm to (59.4, 97.6)
- moved SVI5 0.76 mm to (59.4, 74.7)
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Connections:
- net GND: now also PWR_IN.3; no longer PWR_IN.1
- net N$1: now also PWR_IN.1; no longer PWR_IN.3
Routing:
- net +18V: track 0.00 -> 197.8 mm
- net PA45: track 0.00 -> 75.6 mm
- net PA43: track 0.00 -> 73.7 mm
- net PA29: track 0.00 -> 51.7 mm
- net PA27: track 0.00 -> 44.4 mm
- net PA41: track 0.00 -> 43.0 mm
- net PA39: track 0.00 -> 40.9 mm
- net PA25: track 0.00 -> 33.5 mm
- net PA33: track 0.00 -> 33.3 mm
- net PA47: track 0.00 -> 32.2 mm
- net PA23: track 0.00 -> 31.8 mm
- net PA31: track 0.00 -> 30.7 mm
- net PA37: track 0.00 -> 26.6 mm
- net PA49: track 0.00 -> 25.5 mm
- net PA35: track 0.00 -> 23.4 mm
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Other:
- board text added: "BOTTOM LAYER"
- board text added: "TOP LAYER"
- board text added: "ULTRASONIC MATRIX"
- board text added: "github.com/victorsvi (victorsvi@gmail.com)"

Commit message: more tracing
Parts:
- moved U$30 412.4 mm to (78.5, 134.5), turned to 90 degrees
- moved U$18 405.0 mm to (95.5, 134.5), turned to 90 degrees
- moved U$29 390.6 mm to (78.5, 117.5), turned to 270 degrees
- moved U$17 382.7 mm to (95.5, 117.5), turned to 270 degrees
- moved U$26 354.0 mm to (95.5, 100.5), turned to 90 degrees
- moved U$38 354.0 mm to (78.5, 66.5), turned to 90 degrees
- moved C10 334.6 mm to (133.6, 27.2), turned to 270 degrees
- moved U$37 334.3 mm to (78.5, 49.5), turned to 270 degrees
- moved U$14 332.8 mm to (112.5, 66.5), turned to 90 degrees
- moved U$25 332.5 mm to (95.5, 83.5), turned to 270 degrees
- moved U$13 332.0 mm to (129.0, 66.8)
- moved U$46 305.7 mm to (61.5, 83.5), turned to 270 degrees
- moved U$34 301.5 mm to (78.5, 100.5), turned to 90 degrees
- moved U$45 295.1 mm to (61.5, 100.5), turned to 90 degrees
- moved U$33 280.5 mm to (78.5, 83.5), turned to 270 degrees
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Connections:
- net PA22: now also U9.4; no longer U9.2
- net PA24: now also U9.2; no longer U9.4
- net PA26: now also U11.4; no longer U11.2
- net PA28: now also U11.2; no longer U11.4
- net PA30: now also U13.4; no longer U13.2
- net PA32: now also U13.2; no longer U13.4
- net PA34: now also U15.4; no longer U15.2
- net PA36: now also U15.2; no longer U15.4
- net PA38: now also U17.4; no longer U17.2
- net PA40: now also U17.2; no longer U17.4
- net PA42: now also U19.4; no longer U19.2
- net PA44: now also U19.2; no longer U19.4
- net PA46: now also U21.4; no longer U21.2
- net PA48: now also U21.2; no longer U21.4
- net PA50: now also U23.4; no longer U23.2
- net PA52: now also U23.2; no longer U23.4
- net PD22: now also U$17.P0, U9.5; no longer U$18.P0, U9.7
- net PD24: now also U$18.P0, U9.7; no longer U$17.P0, U9.5
- net PD26: now also U$21.P0, U11.5; no longer U$22.P0, U11.7
- net PD28: now also U$22.P0, U11.7; no longer U$21.P0, U11.5
- net PD30: now also U$25.P0, U13.5; no longer U$26.P0, U13.7
- net PD32: now also U$26.P0, U13.7; no longer U$25.P0, U13.5
- net PD34: now also U$29.P0, U15.5; no longer U$30.P0, U15.7
- net PD36: now also U$30.P0, U15.7; no longer U$29.P0, U15.5
- net PD38: now also U$33.P0, U17.5; no longer U$34.P0, U17.7
- net PD40: now also U$34.P0, U17.7; no longer U$33.P0, U17.5
- net PD42: now also U$37.P0, U19.5; no longer U$38.P0, U19.7
- net PD44: now also U$38.P0, U19.7; no longer U$37.P0, U19.5
- net PD46: now also U$41.P0, U21.5; no longer U$42.P0, U21.7
- net PD48: now also U$42.P0, U21.7; no longer U$41.P0, U21.5
- net PD50: now also U$45.P0, U23.5; no longer U$46.P0, U23.7
- net PD52: now also U$46.P0, U23.7; no longer U$45.P0, U23.5
Routing:
- net +18V: track 197.8 -> 431.2 mm, vias 0 -> 8
- net PA22: track 0.00 -> 81.8 mm
- net PA36: track 0.00 -> 81.7 mm
- net PA34: track 0.00 -> 80.4 mm
- net PA24: track 7.51 -> 84.8 mm
- net PA50: track 0.00 -> 50.9 mm
- net PA51: track 8.48 -> 58.6 mm
- net PA52: track 0.00 -> 49.0 mm
- net PA40: track 0.00 -> 48.5 mm
- net PA30: track 0.00 -> 47.6 mm
- net PA53: track 5.26 -> 52.7 mm
- net PA38: track 0.00 -> 46.6 mm
- net PA32: track 0.00 -> 45.7 mm
- net PD10: track 0.00 -> 30.9 mm
- net GND: track 0.00 -> 19.3 mm, vias 4 -> 6
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Other:
- board size 150 x 150 mm -> 140 x 150 mm

Commit message: almost done
Parts:
- moved U$10 441.9 mm to (95.5, 134.5), turned to 90 degrees
- moved U$9 419.6 mm to (95.5, 117.5), turned to 270 degrees
- moved U$5 399.2 mm to (129.5, 134.5), turned to 180 degrees
- moved U$6 398.8 mm to (112.5, 134.5), turned to 180 degrees
- moved U$8 397.9 mm to (78.5, 134.5), turned to 90 degrees
- moved U$7 375.2 mm to (78.5, 117.5), turned to 270 degrees
- moved U$4 353.4 mm to (112.5, 100.5), turned to 270 degrees
- moved U$60 346.9 mm to (44.5, 66.5), turned to 90 degrees
- moved U$3 346.9 mm to (112.5, 117.5), turned to 270 degrees
- moved U$2 339.2 mm to (129.5, 100.5), turned to 270 degrees
- moved U$1 333.9 mm to (129.5, 117.5), turned to 270 degrees
- moved U$59 328.5 mm to (44.5, 49.5), turned to 270 degrees
- moved U$11 309.1 mm to (129.5, 83.5), flipped to the bottom, turned to 90 degrees
- moved U$12 308.6 mm to (112.5, 83.5), flipped to the bottom, turned to 90 degrees
- moved C8 306.7 mm to (125.5, 50.0), turned to 90 degrees
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Connections:
- net PA6: now also U1.4; no longer U1.2
- net PA64: now also U30.4; no longer U30.2
- net PA65: now also U30.2; no longer U30.4
- net PA66: now also U31.4; no longer U31.2
- net PA67: now also U31.2; no longer U31.4
- net PA68: now also U32.4; no longer U32.2
- net PA69: now also U32.2; no longer U32.4
- net PA7: now also U1.2; no longer U1.4
- net PA8: now also U2.4; no longer U2.2
- net PA9: now also U2.2; no longer U2.4
- net PD6: now also U$3.P0, U1.5; no longer U$4.P0, U1.7
- net PD64: now also U$59.P0, U30.5; no longer U$60.P0, U30.7
- net PD65: now also U$60.P0, U30.7; no longer U$59.P0, U30.5
- net PD66: now also U$61.P0, U31.5; no longer U$62.P0, U31.7
- net PD67: now also U$62.P0, U31.7; no longer U$61.P0, U31.5
- net PD68: now also U$63.P0, U32.5; no longer U$64.P0, U32.7
- net PD69: now also U$64.P0, U32.7; no longer U$63.P0, U32.5
- net PD7: now also U$4.P0, U1.7; no longer U$3.P0, U1.5
- net PD8: now also U$5.P0, U2.5; no longer U$6.P0, U2.7
- net PD9: now also U$6.P0, U2.7; no longer U$5.P0, U2.5
Routing:
- net +18V: track 431.2 -> 774.4 mm, vias 8 -> 17
- net PA69: track 5.59 -> 64.8 mm
- net PA68: track 5.59 -> 64.3 mm
- net PA15: track 5.59 -> 57.8 mm
- net PA14: track 5.59 -> 53.9 mm
- net PA67: track 5.59 -> 51.1 mm
- net PA66: track 5.59 -> 48.1 mm
- net PA10: track 5.59 -> 46.3 mm
- net PA8: track 5.59 -> 44.6 mm
- net PA9: track 5.59 -> 44.4 mm
- net PA11: track 5.59 -> 43.3 mm
- net PA36: track 81.7 -> 113.1 mm
- net PA34: track 80.4 -> 111.8 mm
- net PA22: track 81.8 -> 112.2 mm
- net PA24: track 84.8 -> 114.1 mm
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
Commit message: more on board layout
Parts:
- moved C62 162.1 mm to (25.7, 49.5), turned to 270 degrees
- moved C64 134.4 mm to (11.9, 49.3), turned to 270 degrees
- moved C31 134.2 mm to (23.1, 49.5), turned to 270 degrees
- moved C63 133.4 mm to (14.5, 49.3), turned to 270 degrees
- moved C30 133.4 mm to (28.2, 49.5), turned to 270 degrees
- moved C32 129.9 mm to (9.40, 49.3), turned to 270 degrees
- moved C60 119.8 mm to (32.3, 117.3), turned to 270 degrees
- moved C58 118.1 mm to (22.6, 83.6), turned to 270 degrees
- moved C57 115.3 mm to (25.1, 83.6), turned to 270 degrees
- moved C59 112.3 mm to (8.38, 83.6), turned to 270 degrees
- moved C61 111.5 mm to (17.0, 117.3), turned to 270 degrees
- moved U$50 105.1 mm to (44.5, 100.5)
- moved U$58 96.6 mm to (10.5, 134.5)
- moved U$52 89.6 mm to (27.5, 83.5), turned to 270 degrees
- moved U$51 89.2 mm to (27.5, 100.5)
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Connections:
- net PA56: now also U26.4; no longer U26.2
- net PA57: now also U26.2; no longer U26.4
- net PA58: now also U27.4; no longer U27.2
- net PA59: now also U27.2; no longer U27.4
- net PA60: now also U28.4; no longer U28.2
- net PA61: now also U28.2; no longer U28.4
- net PA62: now also U29.4; no longer U29.2
- net PA63: now also U29.2; no longer U29.4
- net PD56: now also U$51.P0, U26.5; no longer U$52.P0, U26.7
- net PD57: now also U$52.P0, U26.7; no longer U$51.P0, U26.5
- net PD58: now also U$53.P0, U27.5; no longer U$54.P0, U27.7
- net PD59: now also U$54.P0, U27.7; no longer U$53.P0, U27.5
- net PD60: now also U$55.P0, U28.5; no longer U$56.P0, U28.7
- net PD61: now also U$56.P0, U28.7; no longer U$55.P0, U28.5
- net PD62: now also U$57.P0, U29.5; no longer U$58.P0, U29.7
- net PD63: now also U$58.P0, U29.7; no longer U$57.P0, U29.5
Routing:
- net +18V: track 774.4 -> 1196.9 mm, vias 17 -> 21
- net PA61: track 11.5 -> 109.3 mm
- net PA60: track 12.6 -> 108.9 mm
- net PA63: track 26.7 -> 104.4 mm
- net PA62: track 25.5 -> 101.0 mm
- net PA59: track 11.8 -> 51.7 mm
- net PA58: track 12.1 -> 50.0 mm
- net PA57: track 5.59 -> 27.5 mm
- net VIN: track 5.59 -> 26.7 mm
- net PA56: track 5.59 -> 25.0 mm
- net RESET: track 5.59 -> 21.8 mm
- net N$4: track 0.00 -> 15.4 mm
- net PD58: track 0.00 -> 14.6 mm
- net PD56: track 0.00 -> 14.6 mm
- net PD63: track 0.00 -> 13.5 mm
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- added copper zone on layer 1, net GND
Other:
- board text added: "0"
- board text added: "1"
- board text added: "10"
- board text added: "11"
- board text added: "12"
- board text added: "13"
- board text added: "14"
- board text added: "15"
- board text added: "16"
- board text added: "17"
- board text added: "18"
- board text added: "19"
- board text added: "2"
- board text added: "20"
- board text added: "21"
- board text added: "23"
- board text added: "25"
- board text added: "27"
- board text added: "29"
- board text added: "3"
- board text added: "31"
- board text added: "33"
- board text added: "35"
- board text added: "37"
- board text added: "39"
- board text added: "3V3"
- board text added: "4"
- board text added: "41"
- board text added: "43"
- board text added: "45"
- board text added: "47"
- board text added: "49"
- board text added: "5"
- board text added: "51"
- board text added: "53"
- board text added: "54"
- board text added: "55"
- board text added: "56"
- board text added: "57"
- board text added: "58"
- board text added: "59"
- board text added: "5V"
- board text added: "6"
- board text added: "60"
- board text added: "61"
- board text added: "62"
- board text added: "63"
- board text added: "64"
- board text added: "65"
- board text added: "66"
- board text added: "67"
- board text added: "68"
- board text added: "69"
- board text added: "7"
- board text added: "8"
- board text added: "9"
- board text added: "AREF"
- board text added: "GND"
- board text added: "IOREF"
- board text added: "RESET"
- board text added: "SCL"
- board text added: "SDA"
- board text added: "VIN"
- board text added: "VIN_EN"

Commit message: routing completed
Parts:
- moved C20 0.51 mm to (35.1, 10.7)
- moved C32 0.25 mm to (9.65, 49.3)
- moved C63 0.25 mm to (14.7, 49.3)
- moved C64 0.25 mm to (12.2, 49.3)
- moved C52 0.25 mm to (32.5, 10.7)
Routing:
- net +18V: track 1196.9 -> 1391.3 mm, vias 21 -> 22
- net GND: track 23.9 -> 75.2 mm, vias 20 -> 22
- net N$1: track 6.77 -> 11.2 mm
- net PA25: track 42.2 -> 40.7 mm
- net PA23: track 37.9 -> 36.5 mm
- net PA27: track 43.6 -> 42.4 mm
- net PA29: track 42.5 -> 41.6 mm
- added copper zone on layer 16, net GND

Commit message: Board completed
Parts:
- U$8: device ultrasonic:TCT40-16 -> TCT40:TCT40-16
- flipped U$11 to the top
- flipped U$12 to the top
Other:
- board text added: "(1,1)"
- board text added: "(1,2)"
- board text added: "(1,3)"
- board text added: "(1,4)"
- board text added: "(1,5)"
- board text added: "(1,6)"
- board text added: "(1,7)"
- board text added: "(1,8)"
- board text added: "(2,1)"
- board text added: "(2,2)"
- board text added: "(2,3)"
- board text added: "(2,4)"
- board text added: "(2,5)"
- board text added: "(2,6)"
- board text added: "(2,7)"
- board text added: "(2,8)"
- board text added: "(3,1)"
- board text added: "(3,2)"
- board text added: "(3,3)"
- board text added: "(3,4)"
- board text added: "(3,5)"
- board text added: "(3,6)"
- board text added: "(3,7)"
- board text added: "(3,8)"
- board text added: "(4,1)"
- board text added: "(4,2)"
- board text added: "(4,3)"
- board text added: "(4,4)"
- board text added: "(4,5)"
- board text added: "(4,6)"
- board text added: "(4,7)"
- board text added: "(4,8)"
- board text added: "(5,1)"
- board text added: "(5,2)"
- board text added: "(5,3)"
- board text added: "(5,4)"
- board text added: "(5,5)"
- board text added: "(5,6)"
- board text added: "(5,7)"
- board text added: "(5,8)"
- board text added: "(6,1)"
- board text added: "(6,2)"
- board text added: "(6,3)"
- board text added: "(6,4)"
- board text added: "(6,5)"
- board text added: "(6,6)"
- board text added: "(6,7)"
- board text added: "(6,8)"
- board text added: "(7,1)"
- board text added: "(7,2)"
- board text added: "(7,3)"
- board text added: "(7,4)"
- board text added: "(7,5)"
- board text added: "(7,6)"
- board text added: "(7,7)"
- board text added: "(7,8)"
- board text added: "(8,1)"
- board text added: "(8,2)"
- board text added: "(8,3)"
- board text added: "(8,4)"
- board text added: "(8,5)"
- board text added: "(8,6)"
- board text added: "(8,7)"
- board text added: "(8,8)"
- board text added: "06"
- board text added: "07"
- board text added: "08"
- board text added: "09"
- board text added: "19VDC"
- board text added: "22"
- board text added: "24"
- board text added: "26"
- board text added: "28"
- board text added: "30"
- board text added: "32"
- board text added: "34"
- board text added: "36"
- board text added: "38"
- board text added: "40"
- board text added: "42"
- board text added: "44"
- board text added: "46"
- board text added: "48"
- board text added: "50"
- board text added: "52"
- board text removed: "18VDC"
